File: hardware/pcb/exoShield/exoShield.brd (EAGLE design)
At the start: 53.3 x 59.8 mm, 17 parts, among them J1 PHOENIX-1803439, J2 PHOENIX-1803439, J3 PHOENIX-1803426, J4 PHOENIX-1803426, J5 ARDUINO_R3_SHIELD, J6 PHOENIX-1803442, J7 PHOENIX-1803442

Commit message: escon logger debug
Parts:
- moved LED1 18.3 mm to (23.0, 13.5)
- moved LED2 18.3 mm to (23.0, 38.0)
- moved R6 18.1 mm to (19.0, 16.0)
- moved R7 18.1 mm to (19.0, 40.5)
- moved J1 17.6 mm to (27.0, 51.0)
- moved J2 17.6 mm to (26.5, 26.5)
- moved J3 17.6 mm to (40.5, 51.0)
- moved J4 17.6 mm to (40.5, 26.5)
- moved J5 17.6 mm to (0.00, 0.00)
- moved J6 17.6 mm to (13.5, 24.5)
- moved J7 17.6 mm to (13.5, 47.5)
- moved R1 17.6 mm to (34.0, 41.0)
- moved R2 17.6 mm to (33.5, 16.0)
- moved R3 17.6 mm to (45.0, 52.5)
- moved R4 17.6 mm to (45.0, 18.0)
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Routing:
- net N$1: track 18.6 -> 16.6 mm
- net DIR2: track 18.6 -> 17.1 mm
- net DIR1: track 22.9 -> 21.4 mm
- net +5V: track 71.4 -> 72.9 mm
- net VEL1: track 23.3 -> 21.9 mm
- net CUR1: track 22.0 -> 20.8 mm
- net POS1: track 47.4 -> 46.8 mm
- net N$8: track 21.9 -> 21.3 mm
- net N$6: track 5.61 -> 5.08 mm
Other:
- board text added: "UDOO I/O 1.1"
- board text removed: "UDOO I/O 1.0"
