File: hardware/pcb/escon-triple-mobo/escon-triple-mobo.sch (KiCad schematic (older format))
At the start: 66 parts, among them J1 PHOENIX-COMBICON-MCV-4POS, J2 PHOENIX-COMBICON-MCV-2POS, J3 PHOENIX-COMBICON-MCV-4POS, J4 PHOENIX-COMBICON-MCV-4POS, P1 CONN_02X20, P2 CONN_02X04, P3 CONN_02X04, P4 CONN_02X07

Commit message: small changes in hardware files. Prolly just metadata. Updated parameter estimation scripts
Other:
- moved on the sheet: C11, C12, C13, C14, C15, C16, C17, C21, C22, C23, C24, C25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
